Commit message: Drive Robot Gazebo

File: description/robot_core.xacro (robot description, xacro)
@@ -17,5 +17,5 @@
     <link name="base_link">
     </link>
-    <!--CHASIS LINK-->>
+    <!--CHASIS LINK-->
     <joint name="chassis_joint" type="fixed">
         <parent link="base_link"/>
@@ -38,7 +38,10 @@
         </collision>
         <xacro:inertial_box mass="0.5" x="0.25" y="0.15" z="0.035">
-        <origin xyz="0.125 0 0.0175" rpy="0 0 0"/>
-    </xacro:inertial_box>
+            <origin xyz="0.125 0 0.0175" rpy="0 0 0"/>
+        </xacro:inertial_box>
     </link>
+    <gazebo reference="chassis">
+        <material>Gazebo/white</material>
+    </gazebo>
     <!--LEFT WHEEL LINK-->
     <joint name="left_wheel_joint" type="continuous">
@@ -64,4 +67,7 @@
     </xacro:inertial_cylinder>
     </link>
+    <gazebo reference="left_wheel">
+        <material>Gazebo/Blue</material>
+    </gazebo>
     <!--RIGHT WHEEL LINK-->
     <joint name="right_wheel_joint" type="continuous">
@@ -87,4 +93,7 @@
     </xacro:inertial_cylinder>
     </link>
+    <gazebo reference="right_wheel">
+        <material>Gazebo/Blue</material>
+    </gazebo>
     <!--CASTER WHEEL LINK-->
     <joint name="caster_wheel_joint" type="fixed">
@@ -109,3 +118,8 @@
     </xacro:inertial_sphere>
     </link>
+    <gazebo reference="caster_wheel">
+        <material>Gazebo/Black</material>
+        <mu1 value="0.001"/>
+        <mu2 value="0.001"/>
+    </gazebo>
 </robot>

Commit message: Addition of many new things

File: description/robot_core.xacro (robot description, xacro)
@@ -13,4 +13,7 @@
     <material name="black">
         <color rgba="0 0 0 1"/>
+    </material>
+    <material name="red">
+        <color rgba="1 0 0 1"/>
     </material>
     <!--BASE  LINK-->

Commit message: Get real robot working

File: description/robot_core.xacro (robot description, xacro)
@@ -28,18 +28,18 @@
     <link name="chassis">
         <visual>
-            <origin xyz="0.125 0 0.0175" rpy="0 0 0"/>
+            <origin xyz="0.1175 0 0.04" rpy="0 0 0"/>
             <geometry>
-                <box size="0.25 0.15 0.035"/>
+                <box size="0.235 0.15 0.08"/>
             </geometry>
             <material name="white"/>
         </visual>
         <collision>
-            <origin xyz="0.125 0 0.0175" rpy="0 0 0"/>
+            <origin xyz="0.1175 0 0.04" rpy="0 0 0"/>
             <geometry>
-                <box size="0.25 0.15 0.035"/>
+                <box size="0.235 0.15 0.08"/>
             </geometry>
         </collision>
-        <xacro:inertial_box mass="0.5" x="0.25" y="0.15" z="0.035">
-            <origin xyz="0.125 0 0.0175" rpy="0 0 0"/>
+        <xacro:inertial_box mass="0.5" x="0.235" y="0.15" z="0.08">
+            <origin xyz="0.1175 0 0.04" rpy="0 0 0"/>
         </xacro:inertial_box>
     </link>
@@ -57,5 +57,5 @@
         <visual>
             <geometry>
-                <cylinder radius="0.025" length="0.02" />
+                <cylinder radius="0.017" length="0.02" />
             </geometry>
             <material name="blue"/>
@@ -63,8 +63,8 @@
         <collision>
             <geometry>
-                <cylinder radius="0.025" length="0.001" />
+                <cylinder radius="0.034" length="0.001" />
             </geometry>
         </collision>
-        <xacro:inertial_cylinder mass="0.1" length="0.02" radius="0.025">
+        <xacro:inertial_cylinder mass="0.1" length="0.02" radius="0.034">
         <origin xyz="0 0 0" rpy="0 0 0"/>
     </xacro:inertial_cylinder>
@@ -83,5 +83,5 @@
         <visual>
             <geometry>
-                <cylinder radius="0.025" length="0.02" />
+                <cylinder radius="0.034" length="0.02" />
             </geometry>
             <material name="blue"/>
@@ -89,8 +89,8 @@
         <collision>
             <geometry>
-                <cylinder radius="0.025" length="0.001" />
+                <cylinder radius="0.034" length="0.001" />
             </geometry>
         </collision>
-        <xacro:inertial_cylinder mass="0.1" length="0.02" radius="0.025">
+        <xacro:inertial_cylinder mass="0.1" length="0.02" radius="0.034">
         <origin xyz="0 0 0" rpy="0 0 0"/>
     </xacro:inertial_cylinder>

File: description/ros2_control.xacro (robot description, xacro)
@@ -1,5 +1,33 @@
 <?xml version="1.0"?>
 <robot xmlns:xacro="http://www.ros.org/wiki/xacro">
-    <ros2_control name="GazeboSystem" type="system">
+    <ros2_control name="RealRobot" type="system">
+        <hardware>
+            <plugin>diffdrive_arduino/DiffDriveArduino</plugin>
+            <param name="left_wheel_name">left_wheel_joint</param>
+            <param name="right_wheel_name">right_wheel_joint</param>
+            <param name="loop_rate">30</param>
+            <param name="device">/dev/ttyUSB0</param>
+            <param name="baud_rate">57600</param>
+            <param name="timeout">1000</param>
+            <param name="enc_counts_per_rev">1601</param>
+        </hardware>
+        <joint name="left_wheel_joint">
+            <command_interface name="velocity">
+                <param name="min">-10</param>
+                <param name="max">10</param>
+            </command_interface>
+            <state_interface name="velocity"/>
+            <state_interface name="position"/>
+        </joint>
+        <joint name="right_wheel_joint">
+            <command_interface name="velocity">
+                <param name="min">-10</param>
+                <param name="max">10</param>
+            </command_interface>
+            <state_interface name="velocity"/>
+            <state_interface name="position"/>
+        </joint>
+    </ros2_control>
+    <!--ros2_control name="GazeboSystem" type="system">
         <hardware>
             <plugin>gazebo_ros2_control/GazeboSystem</plugin>
@@ -21,5 +49,5 @@
             <state_interface name="position"/>
         </joint>
-    </ros2_control>
+    </ros2_control-->
     <gazebo>
         <plugin name="gazebo_ros2_control" filename="libgazebo_ros2_control.so">

Commit message: Add SLAM stuff

File: description/robot_core.xacro (robot description, xacro)
@@ -19,4 +19,12 @@
     <!--BASE  LINK-->
     <link name="base_link">
+    </link>
+    <!-- BASE_FOOTPRINT LINK -->
+    <joint name="base_footprint_joint" type="fixed">
+        <parent link="base_link"/>
+        <child link="base_footprint"/>
+        <origin xyz="0 0 0" rpy="0 0 0"/>
+    </joint>
+    <link name="base_footprint">
     </link>
     <!--CHASIS LINK-->
